Commit message: Firstm

File: assistive_gym/envs/assets/bed/hospital_bed.urdf (robot description, URDF)
Before this commit: robot bed, 3 links, 2 joints
Links:
- link bottom: geometry collision box size=1 1.25 0.05; visual box size=1 1.25 0.05
- link top: geometry collision box size=1 0.85 0.05; visual box size=1 0.85 0.05
