Commit message: Want_to_train_handover

File: assistive_gym/envs/assets/scratcher/tool_scratch.urdf (robot description, URDF)
Before this commit: robot scratcher, 3 links, 2 joints
Links:
- removed link tool_tip
- link handle: geometry collision cylinder length=0.05 radius=0.01; visual cylinder length=0.10 radius=0.025
- link tool: geometry collision cylinder length=0.005 radius=0.001; visual cylinder length=0.005 radius=0.001
Joints:
- removed joint j_weld2
